File: KiCAD Files/NiCd Battery Shield - VP400KH-REV 1.1/MICROCONTROLLER.sch (KiCad schematic (older format))
At the start: 5 parts, among them SW1 RESET, U4 MEGA_2560_PRO_MINI-NiCd_Batte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

Commit message: Added Rev 1.1 initial commit
Parts:
- removed SW1: RESET, Button_Switch_THT:SW_PUSH_6mm_H5mm, symbol Switch:SW_Push
- added J14: LCD, Connector_PinHeader_2.54mm:PinHeader_1x04_P2.54mm_Vertical, symbol Connector_Generic:Conn_01x04
- added J15: SD CARD, Connector_PinHeader_2.54mm:PinHeader_1x06_P2.54mm_Vertical, symbol Connector_Generic:Conn_01x06
Connections:
- net 5V: now also J14.2 (Pin_2), J15.2 (Pin_2)
- net CS: now also J15.6 (Pin_6)
- net GND: now also J14.1 (Pin_1), J15.1 (Pin_1)
- net MISO: now also J15.3 (Pin_3)
- net MOSI: now also J15.4 (Pin_4)
- net SCK: now also J15.5 (Pin_5)
- net SCL: now also J14.4 (Pin_4)
- net SDA: now also J14.3 (Pin_3)
Changed lines of the file:
@@
 Sheet 3 4
 Title "MICROCONTROLLER"
-Date "2021-04-16"
-Rev "1"
+Date "2021-06-24"
+Rev "1.1"
 Comp ""
 Comment1 ""
@@
 Comment4 ""
 $EndDescr
-$Comp
-L Switch:SW_Push SW?
-U 1 1 607C35A1
-P 4200 2500
-AR Path="/607C35A1" Ref="SW?"  Part="1"
-AR Path="/607B886A/607C35A1" Ref="SW?"  Part="1"
-AR Path="/60829CC7/607C35A1" Ref="SW1"  Part="1"
-F 0 "SW1" H 4200 2785 50  0000 C CNN
-F 1 "RESET" H 4200 2694 50  0000 C CNN
-F 2 "Button_Switch_THT:SW_PUSH_6mm_H5mm" H 4200 2700 50  0001 C CNN
-F 3 "~" H 4200 2700 50  0001 C CNN
-	1    4200 2500
-	1    0    0    -1
-$EndComp
 Text GLabel 4600 4600 0    50   Input ~ 0
 SDA
@@
 Wire Wire Line
 	5900 5300 6000 5300
-$Comp
-L power:GND #PWR?
-U 1 1 607C35E7
-P 3900 2500
-AR Path="/607C35E7" Ref="#PWR?"  Part="1"
-AR Path="/607B886A/607C35E7" Ref="#PWR?"  Part="1"
-AR Path="/60829CC7/607C35E7" Ref="#PWR05"  Part="1"
-F 0 "#PWR05" H 3900 2250 50  0001 C CNN
-F 1 "GND" V 3900 2300 50  0000 C CNN
-F 2 "" H 3900 2500 50  0001 C CNN
-F 3 "" H 3900 2500 50  0001 C CNN
-	1    3900 2500
-	0    1    1    0
-$EndComp
-Wire Wire Line
-	3900 2500 4000 2500
-Wire Wire Line
-	4400 2500 4700 2500
 Wire Wire Line
 	4600 4600 4700 4600
@@
 Wire Wire Line
 	4600 4400 4700 4400
+Wire Wire Line
+	9000 3900 8900 3900
+Wire Wire Line
+	8900 3800 9000 3800
+Wire Wire Line
+	9000 3700 8900 3700
+Wire Wire Line
+	8900 3600 9000 3600
+Wire Wire Line
+	9000 3500 8900 3500
+Wire Wire Line
+	8900 3400 9000 3400
+$Comp
+L power:GND #PWR?
+U 1 1 60C9F7DF
+P 8900 3400
+AR Path="/60C9F7DF" Ref="#PWR?"  Part="1"
+AR Path="/607CEECB/60C9F7DF" Ref="#PWR?"  Part="1"
+AR Path="/6086926A/60C9F7DF" Ref="#PWR?"  Part="1"
+AR Path="/60829CC7/60C9F7DF" Ref="#PWR012"  Part="1"
+F 0 "#PWR012" H 8900 3150 50  0001 C CNN
+F 1 "GND" V 8900 3200 50  0000 C CNN
+F 2 "" H 8900 3400 50  0001 C CNN
+F 3 "" H 8900 3400 50  0001 C CNN
+	1    8900 3400
+	0    1    1    0
+$EndComp
+Text GLabel 8900 3500 0    50   Input ~ 0
+5V
+Text GLabel 8900 3900 0    50   Input ~ 0
+CS
+Text GLabel 8900 3800 0    50   Input ~ 0
+SCK
+Text GLabel 8900 3700 0    50   Input ~ 0
+MOSI
+Text GLabel 8900 3600 0    50   Input ~ 0
+MISO
+Wire Wire Line
+	8900 2750 9000 2750
+Wire Wire Line
+	9000 2850 8900 2850
+Wire Wire Line
+	8900 2950 9000 2950
+Wire Wire Line
+	9000 3050 8900 3050
+Text GLabel 8900 3050 0    50   Input ~ 0
+SCL
+Text GLabel 8900 2950 0    50   Input ~ 0
+SDA
+$Comp
+L power:GND #PWR?
+U 1 1 60C9F7F0
+P 8900 2750
+AR Path="/60C9F7F0" Ref="#PWR?"  Part="1"
+AR Path="/607CEECB/60C9F7F0" Ref="#PWR?"  Part="1"
+AR Path="/6086926A/60C9F7F0" Ref="#PWR?"  Part="1"
+AR Path="/60829CC7/60C9F7F0" Ref="#PWR011"  Part="1"
+F 0 "#PWR011" H 8900 2500 50  0001 C CNN
+F 1 "GND" V 8905 2622 50  0000 R CNN
+F 2 "" H 8900 2750 50  0001 C CNN
+F 3 "" H 8900 2750 50  0001 C CNN
+	1    8900 2750
+	0    1    1    0
+$EndComp
+Text GLabel 8900 2850 0    50   Input ~ 0
+5V
+$Comp
+L Connector_Generic:Conn_01x04 J?
+U 1 1 60C9F7F7
+P 9200 2850
+AR Path="/60C9F7F7" Ref="J?"  Part="1"
+AR Path="/607CEECB/60C9F7F7" Ref="J?"  Part="1"
+AR Path="/6086926A/60C9F7F7" Ref="J?"  Part="1"
+AR Path="/60829CC7/60C9F7F7" Ref="J14"  Part="1"
+F 0 "J14" H 9280 2842 50  0000 L CNN
+F 1 "LCD" H 9280 2751 50  0000 L CNN
+F 2 "Connector_PinHeader_2.54mm:PinHeader_1x04_P2.54mm_Vertical" H 9200 2850 50  0001 C CNN
+F 3 "~" H 9200 2850 50  0001 C CNN
+	1    9200 2850
+	1    0    0    -1
+$EndComp
+$Comp
+L Connector_Generic:Conn_01x06 J?
+U 1 1 60C9F7FD
+P 9200 3600
+AR Path="/60C9F7FD" Ref="J?"  Part="1"
+AR Path="/607CEECB/60C9F7FD" Ref="J?"  Part="1"
+AR Path="/6086926A/60C9F7FD" Ref="J?"  Part="1"
+AR Path="/60829CC7/60C9F7FD" Ref="J15"  Part="1"
+F 0 "J15" H 9150 3900 50  0000 L CNN
+F 1 "SD CARD" V 9300 3400 50  0000 L CNN
+F 2 "Connector_PinHeader_2.54mm:PinHeader_1x06_P2.54mm_Vertical" H 9200 3600 50  0001 C CNN
+F 3 "~" H 9200 3600 50  0001 C CNN
+	1    9200 3600
+	1    0    0    -1
+$EndComp
 $EndSCHEMATC
