File: KiCAD Files/NiCd Battery Shield - VP400KH-REV 1.1/NiCd Battery Shield - VP400KH.kicad_pcb (KiCad board)
At the start: 2 copper layers, 360 x 80 mm, 133 parts, among them J1 Conn_01x01, J10 Conn_01x01, J11 Conn_01x01, J12 Conn_01x01, J13 Conn_01x02, J14 LCD, J15 SD CARD, J2 Conn_01x01, J3 Conn_01x01, J4 Conn_01x01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

Commit message: Added Rev 1.1 initial commit
Parts:
- removed R43, R44: 620R, Resistor_SMD:R_1206_3216Metric_Pad1.42x1.75mm_HandSolder
- added D17: CHARGE STATUS, LED_THT:LED_D5.0mm_Horizontal_O3.81mm_Z3.0mm, F.Cu at (282.8, 187.0)
- added D18: 1N4007, Diode_SMD:D_SMB_Handsoldering, F.Cu at (275.5, 185.5)
- added J16: Conn_01x02, Connector_Molex:Molex_Mini-Fit_Jr_5569-02A2_2x01_P4.20mm_Horizontal, F.Cu at (266.2, 185.5)
- added Q3: 4401, Package_TO_SOT_SMD:SOT-23_Handsoldering, F.Cu at (274.2, 178.5)
- added Q4: 4401, Package_TO_SOT_THT:TO-92L_Inline_Wide, F.Cu at (276.5, 173.5)
- added R51: 620R, Resistor_SMD:R_1206_3216Metric_Pad1.42x1.75mm_HandSolder, F.Cu at (284.2, 183.2)
- added R52: 390R, Resistor_SMD:R_1206_3216Metric_Pad1.42x1.75mm_HandSolder, F.Cu at (280.7, 175.0)
- added R53: 10K, Resistor_SMD:R_1206_3216Metric_Pad1.42x1.75mm_HandSolder, F.Cu at (280.8, 177.5)
- SW1: value RESET -> ON/OFF SWITCH; footprint Button_Switch_THT:SW_PUSH_6mm_H5mm -> NiCd Battery Tester:E_SWITCH_100SP1T1B4M2QE
- moved SW1 104.3 mm to (373.5, 160.5), turned to 180 degrees
- moved C4 3.02 mm to (370.8, 148.5)
- moved J15 0.31 mm to (101.8, 139.2)
- moved J14 0.07 mm to (90.5, 139.5)
Connections:
- F12 pad 2: 12VDC_BUS -> /POWER AND CONTROL/12V_POWER_FUSED
- J14 pad 1: 5V -> GND
- J14 pad 2: GND -> 5V
- J15 pad 1: 5V -> GND
- J15 pad 2: GND -> 5V
- SW1 pad 1: GND -> Net-(SW1-Pad1)
- SW1 pad 2: Net-(SW1-Pad2) -> /POWER AND CONTROL/12V_POWER_FUSED
- U4 pad 10: Net-(SW1-Pad2) -> Net-(U4-Pad10)
- U5 pad 1: Net-(R43-Pad2) -> GND
Routing:
- net Net-(SW1-Pad2): track 130.8 -> 0.00 mm, vias 1 -> 0
- net 12VDC_BUS: track 465.0 -> 517.0 mm
- net Net-(D18-Pad2): track 0.00 -> 39.4 mm
- net /POWER AND CONTROL/12V_POWER_FUSED: track 0.00 -> 12.7 mm
- net Net-(Q3-Pad2): track 0.00 -> 10.8 mm
- net 5V: track 461.1 -> 450.7 mm
- net GND: track 110.0 -> 120.0 mm, vias 39 -> 46
- net Net-(D6-Pad2): track 31.5 -> 39.5 mm
- net Net-(R43-Pad2): track 7.47 -> 0.00 mm
- net /OP-AMPS/CELL1_FUSED: track 118.4 -> 122.2 mm
- net Net-(D17-Pad1): track 0.00 -> 3.75 mm
Other:
- board text added: "10 CELL BATTERY MONITOR FOR USE WITH SAFT VP400KH NiCd BATTERIES DESIGNED BY RILEY GUNN REV 1.1 EFFECTIVE JULY 2021"
- board text added: "BUS CONN"
- board text added: "BUS CONNECT ON = CONNECTED TO BUS"
- board text added: "CHARGE"
- board text removed: "10 CELL BATTERY MONITOR FOR USE WITH SAFT VP400KH NiCd BATTERIES DESIGNED BY RILEY GUNN REV 1.0 EFFECTIVE MAY 2021"
- board text removed: "CHARGE CONTROLLER"
- board text removed: "RESET"
